File: Hardware/KiCAD/LedMatrix.kicad_sch (KiCad schematic)
At the start: 17 parts

Commit message: .
Parts:
- renumbered LED13 to LED?, LED3 to LED?, LED6 to LED?, LED15 to LED?, LED9 to LED?, LED7 to LED?, LED10 to LED?, LED8 to LED?, LED11 to LED?, LED2 to LED?, LED16 to LED?, LED4 to LED?, LED12 to LED?, LED14 to LED?, LED1 to LED?, LED5 to LED?, R1 to R?
Other:
- moved on the sheet: LED?, R?

Commit message: .
Parts:
- gave numbers to parts that had none: 17
Changed lines of the file:
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@@
 		(dnp no)
 		(fields_autoplaced yes)
-		(property "Reference" "#PWR?"
+		(property "Reference" "#PWR026"
 			(at 133.35 73.66 0)
 			(effects
@@
 		(dnp no)
 		(fields_autoplaced yes)
-		(property "Reference" "LED?"
+		(property "Reference" "LED13"
 			(at 62.23 113.03 0)
 			(effects
@@
 		(dnp no)
 		(fields_autoplaced yes)
-		(property "Reference" "#PWR?"
+		(property "Reference" "#PWR023"
 			(at 181.61 36.83 0)
 			(effects
@@
 		(dnp no)
 		(fields_autoplaced yes)
-		(property "Reference" "#PWR?"
+		(property "Reference" "#PWR021"
 			(at 132.08 36.83 0)
 			(effects
@@
 		(dnp no)
 		(fields_autoplaced yes)
-		(property "Reference" "#PWR?"
+		(property "Reference" "#PWR028"
 			(at 234.95 73.66 0)
 			(effects
@@
 		(dnp no)
 		(fields_autoplaced yes)
-		(property "Reference" "#PWR?"
+		(property "Reference" "#PWR09"
 			(at 139.7 71.12 0)
 			(effects
@@
 		(dnp no)
 		(fields_autoplaced yes)
-		(property "Reference" "#PWR?"
+		(property "Reference" "#PWR042"
 			(at 241.3 125.73 0)
 			(effects
@@
 		(dnp no)
 		(fields_autoplaced yes)
-		(property "Reference" "LED?"
+		(property "Reference" "LED3"
 			(at 154.94 24.13 0)
 			(effects
@@
 		(dnp no)
 		(fields_autoplaced yes)
-		(property "Reference" "#PWR?"
+		(property "Reference" "#PWR041"
 			(at 189.23 125.73 0)
 			(effects
@@
 		(dnp no)
 		(fields_autoplaced yes)
-		(property "Reference" "#PWR?"
+		(property "Reference" "#PWR01"
 			(at 45.72 123.19 0)
 			(effects
@@
 		(dnp no)
 		(fields_autoplaced yes)
-		(property "Reference" "LED?"
+		(property "Reference" "LED6"
 			(at 106.68 60.96 0)
 			(effects
@@
 		(dnp no)
 		(fields_autoplaced yes)
-		(property "Reference" "LED?"
+		(property "Reference" "LED15"
 			(at 162.56 113.03 0)
 			(effects
@@
 		(dnp no)
 		(fields_autoplaced yes)
-		(property "Reference" "LED?"
+		(property "Reference" "LED9"
 			(at 60.96 90.17 0)
 			(effects
@@
 		(dnp no)
 		(fields_autoplaced yes)
-		(property "Reference" "#PWR?"
+		(property "Reference" "#PWR019"
 			(at 38.1 34.29 0)
 			(effects
@@
 		(dnp no)
 		(fields_autoplaced yes)
-		(property "Reference" "#PWR?"
+		(property "Reference" "#PWR020"
 			(at 88.9 34.29 0)
 			(effects
@@
 		(dnp no)
 		(fields_autoplaced yes)
-		(property "Reference" "#PWR?"
+		(property "Reference" "#PWR034"
 			(at 87.63 102.87 0)
 			(effects
@@
 		(dnp no)
 		(fields_autoplaced yes)
-		(property "Reference" "#PWR?"
+		(property "Reference" "#PWR036"
 			(at 187.96 102.87 0)
 			(effects
@@
 		(dnp no)
 		(fields_autoplaced yes)
-		(property "Reference" "#PWR?"
+		(property "Reference" "#PWR025"
 			(at 233.68 36.83 0)
 			(effects
@@
 		(dnp no)
 		(fields_autoplaced yes)
-		(property "Reference" "#PWR?"
+		(property "Reference" "#PWR035"
 			(at 138.43 102.87 0)
 			(effects
@@
 		(dnp no)
 		(fields_autoplaced yes)
-		(property "Reference" "#PWR?"
+		(property "Reference" "#PWR040"
 			(at 139.7 125.73 0)
 			(effects
@@
 		(dnp no)
 		(fields_autoplaced yes)
-		(property "Reference" "#PWR?"
+		(property "Reference" "#PWR029"
 			(at 146.05 123.19 0)
 			(effects
@@
 		(dnp no)
 		(fields_autoplaced yes)
-		(property "Reference" "#PWR?"
+		(property "Reference" "#PWR031"
 			(at 95.25 100.33 0)
 			(effects
@@
 		(dnp no)
 		(fields_autoplaced yes)
-		(property "Reference" "LED?"
+		(property "Reference" "LED7"
 			(at 156.21 60.96 0)
 			(effects
@@
 		(dnp no)
 		(fields_autoplaced yes)
-		(property "Reference" "LED?"
+		(property "Reference" "LED10"
 			(at 111.76 90.17 0)
 			(effects
@@
 		(dnp no)
 		(fields_autoplaced yes)
-		(property "Reference" "#PWR?"
+		(property "Reference" "#PWR08"
 			(at 90.17 71.12 0)
 			(effects
@@
 		(dnp no)
 		(fields_autoplaced yes)
-		(property "Reference" "LED?"
+		(property "Reference" "LED8"
 			(at 208.28 60.96 0)
 			(effects
@@
 		(dnp no)
 		(fields_autoplaced yes)
-		(property "Reference" "LED?"
+		(property "Reference" "LED11"
 			(at 161.29 90.17 0)
 			(effects
@@
 		(dnp no)
 		(fields_autoplaced yes)
-		(property "Reference" "#PWR?"
+		(property "Reference" "#PWR010"
 			(at 191.77 71.12 0)
 			(effects
@@
 		(dnp no)
 		(fields_autoplaced yes)
-		(property "Reference" "#PWR?"
+		(property "Reference" "#PWR02"
 			(at 81.28 36.83 0)
 			(effects
@@
 		(dnp no)
 		(fields_autoplaced yes)
-		(property "Reference" "#PWR?"
+		(property "Reference" "#PWR032"
 			(at 144.78 100.33 0)
 			(effects
@@
 		(dnp no)
 		(fields_autoplaced yes)
-		(property "Reference" "#PWR?"
+		(property "Reference" "#PWR030"
 			(at 44.45 100.33 0)
 			(effects
@@
 		(dnp no)
 		(fields_autoplaced yes)
-		(property "Reference" "#PWR?"
+		(property "Reference" "#PWR06"
 			(at 96.52 123.19 0)
 			(effects
@@
 		(dnp no)
 		(fields_autoplaced yes)
-		(property "Reference" "LED?"
+		(property "Reference" "LED2"
 			(at 105.41 24.13 0)
 			(effects
@@
 		(dnp no)
 		(fields_autoplaced yes)
-		(property "Reference" "LED?"
+		(property "Reference" "LED16"
 			(at 214.63 113.03 0)
 			(effects
@@
 		(dnp no)
 		(fields_autoplaced yes)
-		(property "Reference" "#PWR?"
+		(property "Reference" "#PWR033"
 			(at 196.85 100.33 0)
 			(effects
@@
 		(dnp no)
 		(fields_autoplaced yes)
-		(property "Reference" "#PWR?"
+		(property "Reference" "#PWR038"
 			(at 198.12 123.19 0)
 			(effects
@@
 		(dnp no)
 		(fields_autoplaced yes)
-		(property "Reference" "LED?"
+		(property "Reference" "LED4"
 			(at 207.01 24.13 0)
 			(effects
@@
 		(dnp no)
 		(fields_autoplaced yes)
-		(property "Reference" "LED?"
+		(property "Reference" "LED12"
 			(at 213.36 90.17 0)
 			(effects
@@
 		(dnp no)
 		(fields_autoplaced yes)
-		(property "Reference" "LED?"
+		(property "Reference" "LED14"
 			(at 113.03 113.03 0)
 			(effects
@@
 		(dnp no)
 		(fields_autoplaced yes)
-		(property "Reference" "#PWR?"
+		(property "Reference" "#PWR07"
 			(at 39.37 71.12 0)
 			(effects
@@
 		(dnp no)
 		(fields_autoplaced yes)
-		(property "Reference" "#PWR?"
+		(property "Reference" "#PWR039"
 			(at 88.9 125.73 0)
 			(effects
@@
 		(dnp no)
 		(fields_autoplaced yes)
-		(property "Reference" "LED?"
+		(property "Reference" "LED1"
 			(at 54.61 24.13 0)
 			(effects
@@
 		(dnp no)
 		(fields_autoplaced yes)
-		(property "Reference" "#PWR?"
+		(property "Reference" "#PWR024"
 			(at 190.5 34.29 0)
 			(effects
@@
 		(dnp no)
 		(fields_autoplaced yes)
-		(property "Reference" "#PWR?"
+		(property "Reference" "#PWR022"
 			(at 138.43 34.29 0)
 			(effects
@@
 		(dnp no)
 		(fields_autoplaced yes)
-		(property "Reference" "LED?"
+		(property "Reference" "LED5"
 			(at 55.88 60.96 0)
 			(effects
@@
 		(dnp no)
 		(fields_autoplaced yes)
-		(property "Reference" "R?"
+		(property "Reference" "R1"
 			(at 246.38 125.73 90)
 			(effects
@@
 		(dnp no)
 		(fields_autoplaced yes)
-		(property "Reference" "#PWR?"
+		(property "Reference" "#PWR037"
 			(at 240.03 102.87 0)
 			(effects
@@
 		(dnp no)
 		(fields_autoplaced yes)
-		(property "Reference" "#PWR?"
+		(property "Reference" "#PWR011"
 			(at 82.55 73.66 0)
 			(effects
@@
 		(dnp no)
 		(fields_autoplaced yes)
-		(property "Reference" "#PWR?"
+		(property "Reference" "#PWR027"
 			(at 182.88 73.66 0)
 			(effects
